File: eagle/cooler/ps.sch (EAGLE design)
At the start: 18 parts, among them IC5 7812TV, J1 PIN2F061.100, J2 PIN2F061.100, J3 PIN2F061.100, J4 PIN2F061.100, J5 PIN2F061.100, J6 PIN2F061.100, Q1 2N5883, T1 2N3055, T2 2N3055

Commit message: layouts
Parts:
- R1, R2, R3: device rcl:R-US_0207/10 -> rcl:R-US_0207/15
Connections:
- removed net N$2: R4.2
- net TEC1: now also X2-1.KL, X2-3.KL
- net TEC2: now also X2-5.KL
- net VDD: now also R4.2
Other:
- note added: "Fans out"
- note added: "Relay"
- note added: "TEC out"
- moved on the sheet: J2, J6, R4
Changed lines of the file:
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@@
 <part name="J3" library="con-faston" deviceset="PIN2" device="F061.100"/>
 <part name="J4" library="con-faston" deviceset="PIN2" device="F061.100"/>
-<part name="R1" library="rcl" deviceset="R-US_" device="0207/10" value="1K"/>
+<part name="R1" library="rcl" deviceset="R-US_" device="0207/15" value="1K"/>
 <part name="T1" library="transistor" deviceset="2N3055" device=""/>
 <part name="Q1" library="transistor-pnp" deviceset="2N4905" device="" value="2N5883"/>
-<part name="R2" library="rcl" deviceset="R-US_" device="0207/10" value="1.8K"/>
-<part name="R3" library="rcl" deviceset="R-US_" device="0207/10" value="10"/>
+<part name="R2" library="rcl" deviceset="R-US_" device="0207/15" value="1.8K"/>
+<part name="R3" library="rcl" deviceset="R-US_" device="0207/15" value="10"/>
 <part name="R4" library="rcl" deviceset="R-US_" device="0922/22" value="1"/>
 <part name="GND1" library="supply1" deviceset="GND" device=""/>
@@
 <plain>
 <text x="165.1" y="20.32" size="1.778" layer="98">Ultrasonic transducer driver</text>
+<text x="195.58" y="96.52" size="1.778" layer="97">Fans out</text>
+<text x="226.06" y="96.52" size="1.778" layer="97">TEC out</text>
+<text x="162.56" y="142.24" size="1.778" layer="97">Relay</text>
 </plain>
 <instances>
@@
 <instance part="R2" gate="G$1" x="104.14" y="106.68" rot="R90"/>
 <instance part="R3" gate="G$1" x="78.74" y="127"/>
-<instance part="R4" gate="G$1" x="116.84" y="144.78"/>
+<instance part="R4" gate="G$1" x="114.3" y="144.78"/>
 <instance part="GND1" gate="1" x="104.14" y="93.98"/>
 <instance part="VDD1" gate="G$1" x="147.32" y="157.48"/>
 <instance part="J1" gate="-1" x="152.4" y="149.86"/>
-<instance part="J2" gate="-1" x="177.8" y="149.86" rot="R180"/>
+<instance part="J2" gate="-1" x="218.44" y="111.76" rot="R180"/>
 <instance part="J5" gate="-1" x="152.4" y="137.16"/>
-<instance part="J6" gate="-1" x="177.8" y="137.16" rot="R180"/>
+<instance part="J6" gate="-1" x="218.44" y="132.08" rot="R180"/>
 <instance part="X2" gate="-1" x="236.22" y="106.68" rot="R180"/>
 <instance part="X2" gate="-2" x="236.22" y="111.76" rot="R180"/>
@@
 <wire x1="91.44" y1="144.78" x2="104.14" y2="144.78" width="0.1524" layer="91"/>
 <pinref part="R4" gate="G$1" pin="1"/>
-<wire x1="104.14" y1="144.78" x2="111.76" y2="144.78" width="0.1524" layer="91"/>
+<wire x1="104.14" y1="144.78" x2="109.22" y2="144.78" width="0.1524" layer="91"/>
 <pinref part="T2" gate="A" pin="B"/>
 <wire x1="104.14" y1="160.02" x2="104.14" y2="144.78" width="0.1524" layer="91"/>
@@
 <pinref part="R1" gate="G$1" pin="2"/>
 <pinref part="IC5" gate="A1" pin="VO"/>
-<wire x1="127" y1="149.86" x2="127" y2="127" width="0.1524" layer="91"/>
+<wire x1="127" y1="149.86" x2="127" y2="144.78" width="0.1524" layer="91"/>
+<wire x1="127" y1="144.78" x2="127" y2="127" width="0.1524" layer="91"/>
 <wire x1="127" y1="127" x2="127" y2="124.46" width="0.1524" layer="91"/>
 <wire x1="114.3" y1="127" x2="127" y2="127" width="0.1524" layer="91"/>
@@
 <pinref part="T2" gate="A" pin="E"/>
 <wire x1="109.22" y1="165.1" x2="109.22" y2="149.86" width="0.1524" layer="91"/>
+<pinref part="R4" gate="G$1" pin="2"/>
+<wire x1="119.38" y1="144.78" x2="127" y2="144.78" width="0.1524" layer="91"/>
 </segment>
 <segment>
@@
 </segment>
 </net>
-<net name="N$2" class="0">
-<segment>
-<pinref part="R4" gate="G$1" pin="2"/>
-<wire x1="127" y1="144.78" x2="121.92" y2="144.78" width="0.1524" layer="91"/>
-</segment>
-</net>
-<net name="TEC1" class="0">
-<segment>
-<pinref part="J2" gate="-1" pin="1"/>
-<wire x1="182.88" y1="149.86" x2="190.5" y2="149.86" width="0.1524" layer="91"/>
-</segment>
-<segment>
-<wire x1="223.52" y1="116.84" x2="231.14" y2="116.84" width="0.1524" layer="91"/>
-</segment>
-<segment>
-<wire x1="223.52" y1="106.68" x2="231.14" y2="106.68" width="0.1524" layer="91"/>
-</segment>
-</net>
 <net name="TEC2" class="0">
-<segment>
-<pinref part="J6" gate="-1" pin="1"/>
-<wire x1="182.88" y1="137.16" x2="190.5" y2="137.16" width="0.1524" layer="91"/>
-</segment>
 <segment>
 <pinref part="X2" gate="-7" pin="KL"/>
 <wire x1="231.14" y1="137.16" x2="223.52" y2="137.16" width="0.1524" layer="91"/>
-</segment>
-<segment>
 <wire x1="231.14" y1="127" x2="223.52" y2="127" width="0.1524" layer="91"/>
-</segment>
-</net>
+<wire x1="223.52" y1="137.16" x2="223.52" y2="132.08" width="0.1524" layer="91"/>
+<pinref part="J6" gate="-1" pin="1"/>
+<wire x1="223.52" y1="132.08" x2="223.52" y2="127" width="0.1524" layer="91"/>
+<junction x="223.52" y="132.08"/>
+<pinref part="X2" gate="-5" pin="KL"/>
+</segment>
+</net>
+<net name="TEC1" class="0">
+<segment>
+<pinref part="X2" gate="-3" pin="KL"/>
+<pinref part="J2" gate="-1" pin="1"/>
+<wire x1="231.14" y1="116.84" x2="223.52" y2="116.84" width="0.1524" layer="91"/>
+<wire x1="223.52" y1="116.84" x2="223.52" y2="111.76" width="0.1524" layer="91"/>
+<wire x1="223.52" y1="111.76" x2="223.52" y2="106.68" width="0.1524" layer="91"/>
+<pinref part="X2" gate="-1" pin="KL"/>
+<wire x1="223.52" y1="106.68" x2="231.14" y2="106.68" width="0.1524" layer="91"/>
+</segment>
+</net>
