File: eagle/cooler/ps2.brd (EAGLE design)
At the start: 177.8 x 101.6 mm, 18 parts, among them IC5 7812TV, J1 PIN2F061.100, J2 PIN2F061.100, J3 PIN2F061.100, J4 PIN2F061.100, J5 PIN2F061.100, J6 PIN2F061.100, Q1 2N5883, T1 2N3055, T2 2N3055

Commit message: rev2
Routing:
- net GND: track 36.9 -> 0.10 mm
Changed lines of the file:
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@@
 <contactref element="C4" pad="-"/>
 <contactref element="R2" pad="1"/>
-<contactref element="C3" pad="-"/>
-<contactref element="J4" pad="A1"/>
-<contactref element="J4" pad="A2"/>
 <contactref element="X3" pad="2"/>
 <contactref element="X3" pad="4"/>
@@
 <contactref element="X2" pad="6"/>
 <contactref element="X2" pad="8"/>
-<wire x1="3.85" y1="73.66" x2="40.64" y2="73.66" width="2.54" layer="1"/>
 <polygon width="0.6096" layer="1" isolate="1.6764" thermals="no">
 <vertex x="38.1" y="74.93"/>
@@
 <vertex x="1.27" y="76.2"/>
 </polygon>
+<contactref element="C3" pad="-"/>
+<contactref element="J4" pad="A2"/>
+<contactref element="J4" pad="A1"/>
 </signal>
 <signal name="VIN">
