File: eagle/cooler/control_wiring.sch (EAGLE design)
At the start: 7 parts, among them K1 4052, X1 6ESRM-P

Commit message: auber
Parts:
- removed B1: (no value), rectifier:KBL
- removed TR1: (no value), trafo:EI30-1
Changed lines of the file:
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@@
 <part name="P+1" library="supply1" deviceset="VCC" device=""/>
 <part name="X1" library="con-tycoelectronics" deviceset="6ESRM-P" device=""/>
-<part name="TR1" library="trafo" deviceset="EI30-1" device=""/>
-<part name="B1" library="rectifier" deviceset="KBL" device=""/>
 <part name="P+2" library="supply1" deviceset="VCC" device=""/>
 <part name="D2" library="diode" deviceset="1N4004" device=""/>
@@
 <instance part="P+1" gate="VCC" x="99.06" y="83.82" rot="R90"/>
 <instance part="X1" gate="G$1" x="50.8" y="63.5" rot="R270"/>
-<instance part="TR1" gate="1" x="-5.08" y="78.74"/>
-<instance part="B1" gate="1" x="45.72" y="38.1"/>
 <instance part="P+2" gate="VCC" x="99.06" y="55.88" rot="R90"/>
 <instance part="D2" gate="1" x="109.22" y="68.58" rot="R270"/>
