File: eagle/cooler/ps3.sch (EAGLE design)
At the start: 18 parts, among them IC5 7812TV, J1 PIN2F061.100, J2 PIN2F061.100, J3 PIN2F061.100, J4 PIN2F061.100, J5 PIN2F061.100, J6 PIN2F061.100, Q1 2N5883, T1 2N3055, T2 2N3055

Commit message: rev2
Other:
- moved on the sheet: T1, T2
Changed lines of the file:
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@@
 <part name="GND10" library="supply1" deviceset="GND" device=""/>
 <part name="T2" library="transistor" deviceset="2N3055" device=""/>
-<part name="GND11" library="supply1" deviceset="GND" device=""/>
-<part name="GND12" library="supply1" deviceset="GND" device=""/>
 </parts>
 <sheets>
@@
 <instance part="J4" gate="-1" x="22.86" y="101.6" rot="R180"/>
 <instance part="R1" gate="G$1" x="127" y="119.38" rot="R90"/>
-<instance part="T1" gate="A" x="101.6" y="147.32" rot="R90"/>
+<instance part="T1" gate="A" x="104.14" y="147.32" rot="R90"/>
 <instance part="Q1" gate="A" x="86.36" y="142.24" rot="R90"/>
 <instance part="R2" gate="G$1" x="104.14" y="106.68" rot="R90"/>
@@
 <instance part="GND9" gate="1" x="228.6" y="132.08" rot="R270"/>
 <instance part="GND10" gate="1" x="228.6" y="142.24" rot="R270"/>
-<instance part="T2" gate="A" x="101.6" y="157.48" rot="R90"/>
-<instance part="GND11" gate="1" x="66.04" y="99.06"/>
-<instance part="GND12" gate="1" x="30.48" y="99.06"/>
+<instance part="T2" gate="A" x="104.14" y="162.56" rot="R90"/>
 </instances>
 <busses>
@@
 </segment>
 <segment>
+<pinref part="R2" gate="G$1" pin="1"/>
 <pinref part="GND1" gate="1" pin="GND"/>
-<pinref part="R2" gate="G$1" pin="1"/>
 <wire x1="104.14" y1="101.6" x2="104.14" y2="96.52" width="0.1524" layer="91"/>
+<pinref part="C3" gate="G$1" pin="-"/>
+<wire x1="66.04" y1="104.14" x2="66.04" y2="101.6" width="0.1524" layer="91"/>
+<wire x1="27.94" y1="101.6" x2="66.04" y2="101.6" width="0.1524" layer="91"/>
+<wire x1="66.04" y1="101.6" x2="104.14" y2="101.6" width="0.1524" layer="91"/>
+<pinref part="J4" gate="-1" pin="1"/>
 </segment>
 <segment>
@@
 <pinref part="GND10" gate="1" pin="GND"/>
 </segment>
-<segment>
-<pinref part="C3" gate="G$1" pin="-"/>
-<wire x1="66.04" y1="104.14" x2="66.04" y2="101.6" width="0.1524" layer="91"/>
-<pinref part="GND11" gate="1" pin="GND"/>
-</segment>
-<segment>
-<pinref part="J4" gate="-1" pin="1"/>
-<pinref part="GND12" gate="1" pin="GND"/>
-<wire x1="30.48" y1="101.6" x2="27.94" y2="101.6" width="0.1524" layer="91"/>
-</segment>
 </net>
 <net name="VIN" class="0">
@@
 <pinref part="T1" gate="A" pin="C"/>
 <wire x1="66.04" y1="144.78" x2="66.04" y2="149.86" width="0.1524" layer="91"/>
-<wire x1="66.04" y1="149.86" x2="96.52" y2="149.86" width="0.1524" layer="91"/>
+<wire x1="66.04" y1="149.86" x2="99.06" y2="149.86" width="0.1524" layer="91"/>
 <pinref part="Q1" gate="A" pin="E"/>
 <wire x1="66.04" y1="144.78" x2="81.28" y2="144.78" width="0.1524" layer="91"/>
@@
 <pinref part="J3" gate="-1" pin="1"/>
 <pinref part="T2" gate="A" pin="C"/>
-<wire x1="96.52" y1="149.86" x2="96.52" y2="160.02" width="0.1524" layer="91"/>
+<wire x1="99.06" y1="149.86" x2="99.06" y2="165.1" width="0.1524" layer="91"/>
 </segment>
 </net>
@@
 <pinref part="Q1" gate="A" pin="C"/>
 <pinref part="T1" gate="A" pin="B"/>
-<wire x1="91.44" y1="144.78" x2="101.6" y2="144.78" width="0.1524" layer="91"/>
+<wire x1="91.44" y1="144.78" x2="104.14" y2="144.78" width="0.1524" layer="91"/>
 <pinref part="R4" gate="G$1" pin="1"/>
-<wire x1="101.6" y1="144.78" x2="109.22" y2="144.78" width="0.1524" layer="91"/>
+<wire x1="104.14" y1="144.78" x2="109.22" y2="144.78" width="0.1524" layer="91"/>
 <pinref part="T2" gate="A" pin="B"/>
-<wire x1="101.6" y1="154.94" x2="101.6" y2="144.78" width="0.1524" layer="91"/>
+<wire x1="104.14" y1="160.02" x2="104.14" y2="144.78" width="0.1524" layer="91"/>
 </segment>
 </net>
@@
 <wire x1="147.32" y1="154.94" x2="147.32" y2="149.86" width="0.1524" layer="91"/>
 <pinref part="T1" gate="A" pin="E"/>
-<wire x1="106.68" y1="149.86" x2="127" y2="149.86" width="0.1524" layer="91"/>
+<wire x1="109.22" y1="149.86" x2="127" y2="149.86" width="0.1524" layer="91"/>
 <pinref part="R1" gate="G$1" pin="2"/>
 <pinref part="IC5" gate="A1" pin="VO"/>
@@
 <wire x1="147.32" y1="149.86" x2="147.32" y2="137.16" width="0.1524" layer="91"/>
 <pinref part="T2" gate="A" pin="E"/>
-<wire x1="106.68" y1="160.02" x2="106.68" y2="149.86" width="0.1524" layer="91"/>
+<wire x1="109.22" y1="165.1" x2="109.22" y2="149.86" width="0.1524" layer="91"/>
 <pinref part="R4" gate="G$1" pin="2"/>
 <wire x1="119.38" y1="144.78" x2="127" y2="144.78" width="0.1524" layer="91"/>
