File: eagle/cooler/ps3.sch (EAGLE design)
At the start: 19 parts, among them IC5 7812TV, J1 PIN2F061.100, J2 PIN2F061.100, J3 PIN2F061.100, J4 PIN2F061.100, J5 PIN2F061.100, J6 PIN2F061.100, Q1 2N5883, T1 2N3055, T2 2N3055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

Commit message: ps3
Parts:
- removed T2: 2N3055, transistor:2N3055
Connections:
- net B: no longer T2.B
- net VDD: no longer T2.E
- net VIN: no longer T2.C
Changed lines of the file:
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@@
 <part name="GND9" library="supply1" deviceset="GND" device=""/>
 <part name="GND10" library="supply1" deviceset="GND" device=""/>
-<part name="T2" library="transistor" deviceset="2N3055" device=""/>
 <part name="T3" library="transistor" deviceset="2N3055" device=""/>
 </parts>
@@
 <instance part="GND9" gate="1" x="228.6" y="132.08" rot="R270"/>
 <instance part="GND10" gate="1" x="228.6" y="142.24" rot="R270"/>
-<instance part="T2" gate="A" x="104.14" y="167.64" rot="R90"/>
 <instance part="T3" gate="A" x="106.68" y="157.48" rot="R90"/>
 </instances>
@@
 <wire x1="27.94" y1="149.86" x2="66.04" y2="149.86" width="0.1524" layer="91"/>
 <pinref part="J3" gate="-1" pin="1"/>
-<pinref part="T2" gate="A" pin="C"/>
 <wire x1="96.52" y1="149.86" x2="101.6" y2="160.02" width="0.1524" layer="91"/>
 <pinref part="T3" gate="A" pin="C"/>
-<junction x="101.6" y="160.02"/>
-<wire x1="101.6" y1="160.02" x2="99.06" y2="170.18" width="0.1524" layer="91"/>
 </segment>
 </net>
@@
 <pinref part="R4" gate="G$1" pin="1"/>
 <wire x1="101.6" y1="144.78" x2="109.22" y2="144.78" width="0.1524" layer="91"/>
-<pinref part="T2" gate="A" pin="B"/>
 <wire x1="106.68" y1="154.94" x2="101.6" y2="144.78" width="0.1524" layer="91"/>
 <pinref part="T3" gate="A" pin="B"/>
-<junction x="106.68" y="154.94"/>
-<wire x1="106.68" y1="154.94" x2="104.14" y2="165.1" width="0.1524" layer="91"/>
 </segment>
 </net>
@@
 <pinref part="J5" gate="-1" pin="1"/>
 <wire x1="147.32" y1="149.86" x2="147.32" y2="137.16" width="0.1524" layer="91"/>
-<pinref part="T2" gate="A" pin="E"/>
 <wire x1="111.76" y1="160.02" x2="106.68" y2="149.86" width="0.1524" layer="91"/>
 <pinref part="R4" gate="G$1" pin="2"/>
 <wire x1="119.38" y1="144.78" x2="127" y2="144.78" width="0.1524" layer="91"/>
 <pinref part="T3" gate="A" pin="E"/>
-<junction x="111.76" y="160.02"/>
-<wire x1="111.76" y1="160.02" x2="109.22" y2="170.18" width="0.1524" layer="91"/>
 </segment>
 <segment>
