File: eagle/cooler/ps3.brd (EAGLE design)
At the start: 231.1 x 101.6 mm, 19 parts, among them IC5 7812TV, J1 PIN2F061.100, J2 PIN2F061.100, J3 PIN2F061.100, J4 PIN2F061.100, J5 PIN2F061.100, J6 PIN2F061.100, Q1 2N5883, T1 2N3055, T2 2N3055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

Commit message: ps3
Parts:
- removed T2: 2N3055, transistor:TO3
- moved T3 53.3 mm to (26.7, 27.9), turned to 135 degrees
- moved J4 1.27 mm to (5.08, 73.7)
- moved C3 1.27 mm to (74.9, 73.7)
Connections:
- net B: no longer T2.B
- net VDD: no longer T2.E
- net VIN: no longer T2.C, T2.C/
Routing:
- net VDD: track 147.0 -> 481.0 mm, vias 0 -> 1
- net VIN: track 151.2 -> 226.5 mm
- net GND: track 36.9 -> 0.10 mm
- net B: track 196.8 -> 176.9 mm
- added copper zone on layer 1, net GND
- added copper zone on layer 16, net GND
Other:
- board size 231.1 x 101.6 mm -> 177.8 x 101.6 mm

Commit message: final tweaks on ps3
Parts:
- moved J6 9.25 mm to (161.3, 90.2)
- moved J2 9.25 mm to (161.3, 69.8)
- moved X2 8.03 mm to (176.5, 77.5)
- moved X3 7.62 mm to (176.5, 27.9)
- moved Q1 1.27 mm to (134.6, 27.9)
- moved R2 1.27 mm to (40.6, 81.3)
- moved R3 1.27 mm to (52.1, 90.2)
- moved J3 1.27 mm to (6.35, 82.5)
- moved J4 1.27 mm to (6.35, 73.7)
- moved R4 1.27 mm to (25.4, 78.7)
- moved T3 1.27 mm to (27.9, 27.9)
- moved C3 1.27 mm to (76.2, 73.7)
- moved C4 1.27 mm to (115.6, 72.4)
- moved IC5 1.27 mm to (36.8, 95.2)
- moved R1 1.27 mm to (108.0, 95.2)
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Routing:
- net VDD: track 481.0 -> 505.4 mm
- net TEC1: track 76.2 -> 71.1 mm
- net TEC2: track 74.9 -> 71.1 mm
Other:
- board size 177.8 x 101.6 mm -> 184.2 x 101.6 mm
