File: eagle/disruptor/generator.brd (EAGLE design)
At the start: 160 x 100 mm, 29 parts, among them IC1 NE555, IC2 74ALS04N, IC3 IR2110, IC4 7805TV, J1 PIN2F061.100, J2 PIN2F061.100, J3 PIN2F061.100, J4 PIN2F061.100, J5 PIN2F061.100, J6 PIN2F061.100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

Commit message: layouts
Parts:
- removed R1: (no value), rcl:0207/10
- added C3: 10n, rcl:C075-052X106
- C1, C2: value 2u2 -> .1u; device rcl:EB20D -> rcl:E5-8,5
- C4, C5, C7, C8: value 2u2 -> 1u; device rcl:EB20D -> rcl:E5-8,5
- C6: value 100n -> 10n; device rcl:C150-064X183 -> rcl:C075-052X106
- moved J5 233.5 mm to (120.7, 71.1)
- moved J6 212.5 mm to (120.7, 5.08)
- moved J1 209.5 mm to (118.1, 47.0)
- moved J2 208.0 mm to (118.1, 31.8)
- moved R7 204.1 mm to (102.9, 10.2), turned to 270 degrees
- moved R6 189.7 mm to (86.4, 16.5), turned to 180 degrees
- moved Q2 189.2 mm to (115.6, 21.6)
- moved R4 171.5 mm to (101.6, 34.3), turned to 180 degrees
- moved Q1 170.8 mm to (118.1, 61.0)
- moved R5 167.1 mm to (72.4, 7.62), turned to 90 degrees
- moved S1 164.1 mm to (90.2, 59.7), turned to 90 degrees
- moved C7 161.4 mm to (90.2, 26.7), turned to 180 degrees
- moved D1 143.4 mm to (80.0, 10.2), turned to 180 degrees
- moved J4 134.8 mm to (7.62, 67.3)
- moved IC3 133.5 mm to (87.6, 44.5)
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Connections:
- net N$15 renamed TRANS2
- net N$5 renamed LO
- net N$6 renamed TRANS1
- net N$8 renamed HO
- removed net N$4: IC1.3, IC2.1, IC3.10, R1.1
- new net HIN: IC1.3, IC2.1, IC3.10
- new net LIN: IC2.2, IC3.12
- new net N$10: B1.AC1, J3.A1, J3.A2
- new net N$3: C3.2, IC1.5
- net GND: now also C3.1, C6.1; no longer C6.2
- net N$9: now also B1.AC2, J4.A1, J4.A2; no longer C2.+, IC1.4, R3.E
- net VCC: now also C2.+, C6.2, IC1.4, R3.E; no longer C6.1, R1.2
Other:
- board size 160 x 100 mm -> 127 x 76.2 mm

Commit message: layouts
Parts:
- D1: device diode:D-5 -> diode:D-7.5
- moved J5 122.2 mm to (8.89, 21.6)
- moved J6 111.8 mm to (8.89, 5.08)
- moved Q1 100.7 mm to (25.4, 21.6), turned to 270 degrees
- moved Q2 82.5 mm to (34.3, 7.62), turned to 90 degrees
- moved R7 80.2 mm to (22.9, 5.08), turned to 180 degrees
- moved D1 77.7 mm to (64.8, 86.4), turned to 0 degrees
- moved C7 60.6 mm to (57.1, 77.5), turned to 0 degrees
- moved R4 57.4 mm to (44.5, 29.2), turned to 0 degrees
- moved J2 56.9 mm to (68.6, 3.81)
- moved C3 55.3 mm to (36.8, 58.4), turned to 90 degrees
- moved C2 55.1 mm to (8.89, 53.3), turned to 270 degrees
- moved J1 55.1 mm to (68.6, 22.9), turned to 180 degrees
- moved R2 54.7 mm to (36.8, 77.5), turned to 180 degrees
- moved R6 52.6 mm to (34.3, 24.1), turned to 270 degrees
- moved IC2 49.3 mm to (17.8, 41.9), turned to 180 degrees
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Routing:
- net VDD: track 0.00 -> 88.3 mm
- net HO: track 0.00 -> 81.1 mm
- net LO: track 0.00 -> 61.2 mm
- net LIN: track 0.00 -> 54.0 mm
- net HIN: track 0.00 -> 52.1 mm
- net TRANS1: track 0.00 -> 42.2 mm
- net VCC: track 0.00 -> 30.0 mm
- net N$2: track 0.00 -> 29.6 mm
- net TRANS2: track 0.00 -> 29.5 mm
- net N$1: track 0.00 -> 24.2 mm
- net N$11: track 0.00 -> 24.1 mm
- net N$12: track 0.00 -> 19.9 mm
- net N$9: track 0.00 -> 19.1 mm
- net N$10: track 0.00 -> 18.6 mm
- net N$17: track 0.00 -> 15.2 mm
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- added copper zone on layer 16, net GND
- added copper zone on layer 1, net N$13
- added copper zone on layer 1, net TRANS1
- added copper zone on layer 1, net TRANS2
Other:
- board size 127 x 76.2 mm -> 76.2 x 120.7 mm

Commit message: layouts
Parts:
- R2, R3: device pot:LI15 -> pot:LI10
- moved C1 1.27 mm to (7.62, 64.8)
- moved C2 1.27 mm to (7.62, 53.3), turned to 180 degrees
Routing:
- net VCC: track 30.0 -> 59.3 mm
Changed lines of the file:
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@@
 <element name="IC4" library="linear" package="TO220V" value="7805TV" x="29.21" y="107.95" rot="R90"/>
 <element name="B1" library="rectifier" package="GBU4" value="RECTIFIER-GBU4" x="20.32" y="106.68" rot="R270"/>
-<element name="R2" library="pot" package="LI15" value="" x="36.83" y="77.47" rot="R180"/>
-<element name="R3" library="pot" package="LI15" value="" x="19.05" y="77.47" rot="R180"/>
-<element name="C1" library="rcl" package="E5-8,5" value=".1u" x="8.89" y="64.77" rot="R180"/>
-<element name="C2" library="rcl" package="E5-8,5" value=".1u" x="8.89" y="53.34" rot="R270"/>
+<element name="R2" library="pot" package="LI10" value="" x="36.83" y="77.47" rot="R180"/>
+<element name="R3" library="pot" package="LI10" value="" x="19.05" y="77.47" rot="R180"/>
+<element name="C1" library="rcl" package="E5-8,5" value=".1u" x="7.62" y="64.77" rot="R180"/>
+<element name="C2" library="rcl" package="E5-8,5" value=".1u" x="7.62" y="53.34" rot="R180"/>
 <element name="Q1" library="transistor-power" package="TO220BV" value="STP11NM60" x="25.4" y="21.59" rot="R270"/>
 <element name="Q2" library="transistor-power" package="TO220BV" value="STP11NM60" x="34.29" y="7.62" rot="R90"/>
@@
 <wire x1="29.21" y1="110.49" x2="26.67" y2="107.95" width="1.6764" layer="1"/>
 <wire x1="26.67" y1="107.95" x2="26.67" y2="90.17" width="1.6764" layer="1"/>
-<wire x1="58.2168" y1="48.26" x2="57.15" y2="60.96" width="0" layer="19" extent="1-1"/>
+<wire x1="57.15" y1="60.96" x2="57.15" y2="59.69" width="1.6764" layer="16"/>
+<wire x1="57.15" y1="60.96" x2="57.15" y2="64.77" width="1.6764" layer="16"/>
+<wire x1="57.15" y1="64.77" x2="48.26" y2="64.77" width="1.6764" layer="16"/>
+<wire x1="26.67" y1="90.17" x2="13.97" y2="90.17" width="1.6764" layer="1"/>
+<wire x1="13.97" y1="90.17" x2="13.97" y2="87.63" width="1.6764" layer="1"/>
+<wire x1="58.2168" y1="48.26" x2="57.15" y2="59.69" width="0" layer="19" extent="16-16"/>
 <wire x1="58.42" y1="40.64" x2="58.2168" y2="48.26" width="0" layer="19" extent="1-1"/>
-<wire x1="26.67" y1="53.34" x2="57.15" y2="60.96" width="0" layer="19" extent="1-1"/>
+<wire x1="26.67" y1="53.34" x2="48.26" y2="64.77" width="0" layer="19" extent="16-16"/>
 <wire x1="19.05" y1="60.96" x2="26.67" y2="53.34" width="0" layer="19" extent="1-1"/>
-<wire x1="8.89" y1="55.88" x2="19.05" y2="60.96" width="0" layer="19" extent="1-1"/>
+<wire x1="10.16" y1="53.34" x2="19.05" y2="60.96" width="0" layer="19" extent="1-1"/>
 <wire x1="25.4" y1="38.1" x2="26.67" y2="53.34" width="0" layer="19" extent="1-1"/>
-<wire x1="13.97" y1="85.09" x2="19.05" y2="60.96" width="0" layer="19" extent="1-1"/>
-<wire x1="26.67" y1="90.17" x2="13.97" y2="85.09" width="0" layer="19" extent="1-1"/>
+<wire x1="16.51" y1="82.55" x2="19.05" y2="60.96" width="0" layer="19" extent="1-1"/>
+<wire x1="13.97" y1="87.63" x2="16.51" y2="82.55" width="0" layer="19" extent="1-1"/>
 </signal>
 <signal name="N$1">
@@
 <wire x1="24.13" y1="64.77" x2="31.75" y2="72.39" width="1.6764" layer="1"/>
 <wire x1="31.75" y1="72.39" x2="36.83" y2="72.39" width="1.6764" layer="1"/>
-<wire x1="36.83" y1="72.39" x2="41.91" y2="85.09" width="0" layer="19" extent="1-1"/>
+<wire x1="36.83" y1="72.39" x2="39.37" y2="82.55" width="0" layer="19" extent="1-1"/>
 <wire x1="21.59" y1="53.34" x2="21.59" y2="52.07" width="0" layer="19" extent="1-1"/>
-<wire x1="11.43" y1="64.77" x2="24.13" y2="64.77" width="0" layer="19" extent="1-1"/>
+<wire x1="10.16" y1="64.77" x2="24.13" y2="64.77" width="0" layer="19" extent="1-1"/>
 </signal>
 <signal name="N$7">
@@
 <wire x1="21.59" y1="60.96" x2="21.59" y2="59.69" width="1.6764" layer="1"/>
 <wire x1="21.59" y1="60.96" x2="21.59" y2="72.39" width="1.6764" layer="1"/>
-<wire x1="24.13" y1="85.09" x2="31.75" y2="85.09" width="0" layer="19" extent="1-1"/>
-<wire x1="21.59" y1="72.39" x2="24.13" y2="85.09" width="0" layer="19" extent="1-1"/>
+<wire x1="21.59" y1="82.55" x2="34.29" y2="82.55" width="0" layer="19" extent="1-1"/>
+<wire x1="21.59" y1="72.39" x2="21.59" y2="82.55" width="0" layer="19" extent="1-1"/>
 <wire x1="19.05" y1="72.39" x2="21.59" y2="72.39" width="0" layer="19" extent="1-1"/>
 </signal>

Commit message: layouts
Parts:
- S1: value (none) -> TL32PO; device switch:320-916 -> switch:TL3XPO
- moved C4 4.82 mm to (42.2, 104.9)
- moved C3 3.94 mm to (35.8, 62.2), turned to 180 degrees
- moved S1 3.81 mm to (58.4, 48.3), turned to 180 degrees
- moved C6 2.55 mm to (59.7, 40.4)
- moved R3 2.54 mm to (21.6, 77.5)
- moved J2 1.78 mm to (68.6, 5.59)
- moved C5 1.55 mm to (39.6, 114.6)
- moved J1 1.55 mm to (68.3, 21.3)
- moved C7 1.27 mm to (55.9, 77.5)
- moved C8 1.27 mm to (67.3, 78.7)
- moved D1 1.27 mm to (63.5, 86.4)
- moved IC3 1.27 mm to (61.0, 64.8)
- moved C2 1.02 mm to (7.62, 54.4)
- moved Q1 0.76 mm to (26.2, 21.6)
- moved J4 0.36 mm to (7.87, 115.8)
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Routing:
- net GND: track 12.3 -> 190.0 mm
- net VCC: track 59.3 -> 228.9 mm
- net TRANS1: track 42.2 -> 201.4 mm
- net TRANS2: track 29.5 -> 114.5 mm
- net N$13: track 10.2 -> 62.5 mm
- net N$9: track 19.1 -> 60.0 mm
- net N$10: track 18.6 -> 54.8 mm
- net N$2: track 29.6 -> 58.6 mm
- net N$7: track 12.7 -> 34.1 mm
- net N$3: track 12.7 -> 7.87 mm
- net HO: track 81.1 -> 77.5 mm
- net HIN: track 52.1 -> 54.4 mm
- net LIN: track 54.0 -> 55.5 mm
- net LO: track 61.2 -> 60.3 mm
- net VDD: track 88.3 -> 87.5 mm
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- removed copper zone on layer 1, net N$13
- removed copper zone on layer 1, net TRANS1
- removed copper zone on layer 1, net TRANS2
