File: eagle/disruptor/generator.sch (EAGLE design)
At the start: 32 parts, among them IC1 NE555, IC2 74ALS04N, IC3 IR2110, IC4 7805TV, IC5 7812TV, J1 PIN2F061.100, J2 PIN2F061.100, J3 PIN2F061.100, J4 PIN2F061.100, J5 PIN2F061.100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

Commit message: change power on gen board
change power on gen board
Parts:
- removed B2: RECTIFIER-GBU4, rectifier:RECTIFIER-GBU4
- removed C3: 2u2, rcl:CPOL-EUE10-20
- removed IC5: 7812TV, linear:7812TV
Connections:
- removed net N$10: B1.+, C3.+, IC5.VI
- removed net N$14: B2.AC2, J6.1
- removed net N$3: B2.AC1, J5.1
- net GND: now also J6.1; no longer B2.+, C3.-, IC5.GND
- net N$13: now also J5.1; no longer B2.-
- net VDD: now also B1.+; no longer IC5.VO
Other:
- moved on the sheet: J5, J6
Changed lines of the file:
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@@
 <part name="IC2" library="74xx-us" deviceset="74*04" device="N" technology="ALS"/>
 <part name="IC4" library="linear" deviceset="78*" device="TV" technology="05"/>
-<part name="IC5" library="linear" deviceset="78*" device="TV" technology="12"/>
 <part name="B1" library="rectifier" deviceset="RECTIFIER-" device="GBU4"/>
 <part name="R1" library="rcl" deviceset="R-US_" device="0207/10"/>
@@
 <part name="Q1" library="transistor-power" deviceset="IRF530" device="" value="STP11NM60"/>
 <part name="Q2" library="transistor-power" deviceset="IRF530" device="" value="STP11NM60"/>
-<part name="C3" library="rcl" deviceset="CPOL-EU" device="E10-20" value="2u2"/>
 <part name="C4" library="rcl" deviceset="CPOL-EU" device="E10-20" value="2u2"/>
 <part name="C5" library="rcl" deviceset="CPOL-EU" device="E10-20" value="2u2"/>
@@
 <part name="J5" library="con-faston" deviceset="PIN2" device="F061.100"/>
 <part name="J6" library="con-faston" deviceset="PIN2" device="F061.100"/>
-<part name="B2" library="rectifier" deviceset="RECTIFIER-" device="GBU4"/>
 <part name="VDD1" library="supply1" deviceset="VDD" device=""/>
 <part name="P+1" library="supply1" deviceset="VCC" device=""/>
@@
 <instance part="IC2" gate="A" x="142.24" y="78.74"/>
 <instance part="IC4" gate="A1" x="127" y="157.48"/>
-<instance part="IC5" gate="A1" x="83.82" y="157.48"/>
 <instance part="B1" gate="G$1" x="25.4" y="154.94"/>
 <instance part="R1" gate="G$1" x="132.08" y="88.9" rot="R90"/>
@@
 <instance part="Q1" gate="G$1" x="231.14" y="91.44"/>
 <instance part="Q2" gate="G$1" x="231.14" y="66.04"/>
-<instance part="C3" gate="G$1" x="58.42" y="154.94" smashed="yes">
-<attribute name="NAME" x="60.7506" y="153.7168" size="1.27" layer="95"/>
-<attribute name="VALUE" x="60.9571" y="151.79" size="1.27" layer="96"/>
-</instance>
 <instance part="C4" gate="G$1" x="106.68" y="154.94" smashed="yes">
 <attribute name="NAME" x="109.0106" y="153.7168" size="1.27" layer="95"/>
@@
 <attribute name="VALUE" x="149.8571" y="151.79" size="1.27" layer="96"/>
 </instance>
-<instance part="GND8" gate="1" x="106.68" y="142.24"/>
+<instance part="GND8" gate="1" x="106.68" y="144.78"/>
 <instance part="R4" gate="G$1" x="220.98" y="88.9" rot="R180"/>
 <instance part="R5" gate="G$1" x="220.98" y="63.5" rot="R180"/>
@@
 <instance part="J3" gate="-1" x="10.16" y="160.02" rot="R180"/>
 <instance part="J4" gate="-1" x="10.16" y="149.86" rot="R180"/>
-<instance part="J5" gate="-1" x="12.7" y="104.14" rot="R180"/>
-<instance part="J6" gate="-1" x="12.7" y="93.98" rot="R180"/>
-<instance part="B2" gate="G$1" x="25.4" y="99.06"/>
+<instance part="J5" gate="-1" x="12.7" y="106.68" rot="R180"/>
+<instance part="J6" gate="-1" x="12.7" y="50.8" rot="R180"/>
 <instance part="VDD1" gate="G$1" x="203.2" y="81.28"/>
 <instance part="P+1" gate="VCC" x="162.56" y="71.12"/>
 <instance part="P+4" gate="VCC" x="177.8" y="101.6"/>
-<instance part="P+3" gate="VCC" x="147.32" y="160.02"/>
+<instance part="P+3" gate="VCC" x="147.32" y="162.56"/>
 <instance part="VDD2" gate="G$1" x="106.68" y="162.56"/>
 <instance part="R6" gate="G$1" x="226.06" y="81.28" rot="R270"/>
@@
 </segment>
 <segment>
+<pinref part="C5" gate="G$1" pin="+"/>
+<pinref part="P+3" gate="VCC" pin="VCC"/>
+<wire x1="147.32" y1="160.02" x2="147.32" y2="157.48" width="0.1524" layer="91"/>
 <pinref part="IC4" gate="A1" pin="VO"/>
-<pinref part="C5" gate="G$1" pin="+"/>
 <wire x1="137.16" y1="157.48" x2="147.32" y2="157.48" width="0.1524" layer="91"/>
-<pinref part="P+3" gate="VCC" pin="VCC"/>
-<junction x="147.32" y="157.48"/>
 </segment>
 </net>
@@
 </segment>
 <segment>
-<pinref part="IC5" gate="A1" pin="VO"/>
 <pinref part="C4" gate="G$1" pin="+"/>
-<wire x1="93.98" y1="157.48" x2="106.68" y2="157.48" width="0.1524" layer="91"/>
 <wire x1="106.68" y1="160.02" x2="106.68" y2="157.48" width="0.1524" layer="91"/>
 <pinref part="IC4" gate="A1" pin="VI"/>
 <wire x1="106.68" y1="157.48" x2="116.84" y2="157.48" width="0.1524" layer="91"/>
 <pinref part="VDD2" gate="G$1" pin="VDD"/>
+<pinref part="B1" gate="G$1" pin="+"/>
+<wire x1="30.48" y1="157.48" x2="30.48" y2="154.94" width="0.1524" layer="91"/>
+<wire x1="30.48" y1="157.48" x2="106.68" y2="157.48" width="0.1524" layer="91"/>
 </segment>
 </net>
@@
 <pinref part="GND1" gate="1" pin="GND"/>
 <wire x1="210.82" y1="66.04" x2="210.82" y2="50.8" width="0.1524" layer="91"/>
-<pinref part="B2" gate="G$1" pin="+"/>
-<wire x1="30.48" y1="99.06" x2="30.48" y2="50.8" width="0.1524" layer="91"/>
 <pinref part="Q2" gate="G$1" pin="S"/>
-<wire x1="30.48" y1="50.8" x2="210.82" y2="50.8" width="0.1524" layer="91"/>
+<wire x1="17.78" y1="50.8" x2="210.82" y2="50.8" width="0.1524" layer="91"/>
 <pinref part="R7" gate="G$1" pin="2"/>
-<wire x1="210.82" y1="50.8" x2="226.06" y2="50.8" width="0.1524" layer="91"/>
 <wire x1="233.68" y1="50.8" x2="233.68" y2="60.96" width="0.1524" layer="91"/>
 <wire x1="226.06" y1="50.8" x2="233.68" y2="50.8" width="0.1524" layer="91"/>
@@
 <pinref part="GND6" gate="1" pin="GND"/>
 <junction x="210.82" y="50.8"/>
+<pinref part="J6" gate="-1" pin="1"/>
 </segment>
 <segment>
@@
 <pinref part="C4" gate="G$1" pin="-"/>
 <wire x1="127" y1="149.86" x2="106.68" y2="149.86" width="0.1524" layer="91"/>
-<pinref part="IC5" gate="A1" pin="GND"/>
-<wire x1="106.68" y1="149.86" x2="83.82" y2="149.86" width="0.1524" layer="91"/>
-<pinref part="C3" gate="G$1" pin="-"/>
-<wire x1="83.82" y1="149.86" x2="58.42" y2="149.86" width="0.1524" layer="91"/>
-<wire x1="58.42" y1="149.86" x2="35.56" y2="149.86" width="0.1524" layer="91"/>
-<wire x1="35.56" y1="149.86" x2="35.56" y2="144.78" width="0.1524" layer="91"/>
-<wire x1="35.56" y1="144.78" x2="17.78" y2="144.78" width="0.1524" layer="91"/>
+<wire x1="106.68" y1="149.86" x2="30.48" y2="144.78" width="0.1524" layer="91"/>
+<wire x1="30.48" y1="144.78" x2="17.78" y2="144.78" width="0.1524" layer="91"/>
 <wire x1="17.78" y1="144.78" x2="17.78" y2="154.94" width="0.1524" layer="91"/>
 <pinref part="B1" gate="G$1" pin="-"/>
 <wire x1="17.78" y1="154.94" x2="20.32" y2="154.94" width="0.1524" layer="91"/>
 <pinref part="GND8" gate="1" pin="GND"/>
-<wire x1="106.68" y1="144.78" x2="106.68" y2="149.86" width="0.1524" layer="91"/>
+<wire x1="106.68" y1="147.32" x2="106.68" y2="149.86" width="0.1524" layer="91"/>
 </segment>
 <segment>
@@
 </segment>
 </net>
-<net name="N$10" class="0">
-<segment>
-<pinref part="B1" gate="G$1" pin="+"/>
-<pinref part="IC5" gate="A1" pin="VI"/>
-<pinref part="C3" gate="G$1" pin="+"/>
-<wire x1="58.42" y1="157.48" x2="73.66" y2="157.48" width="0.1524" layer="91"/>
-<wire x1="58.42" y1="157.48" x2="38.1" y2="157.48" width="0.1524" layer="91"/>
-<wire x1="38.1" y1="157.48" x2="38.1" y2="162.56" width="0.1524" layer="91"/>
-<wire x1="38.1" y1="162.56" x2="30.48" y2="162.56" width="0.1524" layer="91"/>
-<wire x1="30.48" y1="162.56" x2="30.48" y2="154.94" width="0.1524" layer="91"/>
-</segment>
-</net>
 <net name="N$11" class="0">
 <segment>
@@
 </segment>
 </net>
-<net name="N$3" class="0">
-<segment>
+<net name="N$13" class="0">
+<segment>
+<pinref part="Q1" gate="G$1" pin="D"/>
+<wire x1="17.78" y1="106.68" x2="233.68" y2="106.68" width="0.1524" layer="91"/>
+<wire x1="233.68" y1="106.68" x2="233.68" y2="96.52" width="0.1524" layer="91"/>
 <pinref part="J5" gate="-1" pin="1"/>
-<pinref part="B2" gate="G$1" pin="AC1"/>
-<wire x1="17.78" y1="104.14" x2="25.4" y2="104.14" width="0.1524" layer="91"/>
-</segment>
-</net>
-<net name="N$14" class="0">
-<segment>
-<pinref part="J6" gate="-1" pin="1"/>
-<pinref part="B2" gate="G$1" pin="AC2"/>
-<wire x1="25.4" y1="93.98" x2="17.78" y2="93.98" width="0.1524" layer="91"/>
-</segment>
-</net>
-<net name="N$13" class="0">
-<segment>
-<pinref part="B2" gate="G$1" pin="-"/>
-<wire x1="20.32" y1="99.06" x2="20.32" y2="109.22" width="0.1524" layer="91"/>
-<pinref part="Q1" gate="G$1" pin="D"/>
-<wire x1="20.32" y1="109.22" x2="233.68" y2="106.68" width="0.1524" layer="91"/>
-<wire x1="233.68" y1="106.68" x2="233.68" y2="96.52" width="0.1524" layer="91"/>
-</segment>
-</net>
+</segment>
+</net>

Commit message: layouts
Parts:
- removed R1: (no value), rcl:R-US_0207/10
- added C3: 10n, rcl:C-EU075-052X106
- C1, C2: value 2u2 -> .1u; device rcl:CPOL-EUE10-20 -> rcl:CPOL-EUE5-8.5
- C4, C5, C7, C8: value 2u2 -> 1u; device rcl:CPOL-EUE10-20 -> rcl:CPOL-EUE5-8.5
- C6: value 100n -> 10n; device rcl:C-EU150-064X183 -> rcl:C-EU075-052X106
Connections:
- net N$15 renamed TRANS2
- net N$5 renamed LO
- net N$6 renamed TRANS1
- net N$8 renamed HO
- removed net N$4: IC1.OUT, IC2A.I, IC3.10, R1.1
- new net HIN: IC1.OUT, IC2A.I, IC3.10
- new net LIN: IC2A.O, IC3.12
- new net N$10: B1.AC1, J3.1
- new net N$3: C3.2, IC1.CON
- net GND: now also C3.1, C6.1; no longer C6.2
- net N$9: now also B1.AC2, J4.1; no longer C2.+, IC1./RES, R3.E
- net VCC: now also C2.+, C6.2, IC1./RES, R3.E; no longer C6.1, R1.2
Other:
- note added: "12 VAC in"
- note added: "Rectified variac out"
- note added: "Trimmers 500"
- moved on the sheet: C2, C6, J2, J4, J5

Commit message: layouts
Parts:
- D1: device diode:DIODE-D-5 -> diode:DIODE-D-7.5
Changed lines of the file:
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@@
 <grid distance="0.1" unitdist="inch" unit="inch" style="lines" multiple="1" display="no" altdistance="0.01" altunitdist="inch" altunit="inch"/>
 <layers>
-<layer number="1" name="Top" color="4" fill="1" visible="no" active="no"/>
-<layer number="2" name="Route2" color="1" fill="3" visible="no" active="no"/>
-<layer number="3" name="Route3" color="4" fill="3" visible="no" active="no"/>
-<layer number="4" name="Route4" color="1" fill="4" visible="no" active="no"/>
-<layer number="5" name="Route5" color="4" fill="4" visible="no" active="no"/>
-<layer number="6" name="Route6" color="1" fill="8" visible="no" active="no"/>
-<layer number="7" name="Route7" color="4" fill="8" visible="no" active="no"/>
-<layer number="8" name="Route8" color="1" fill="2" visible="no" active="no"/>
-<layer number="9" name="Route9" color="4" fill="2" visible="no" active="no"/>
-<layer number="10" name="Route10" color="1" fill="7" visible="no" active="no"/>
-<layer number="11" name="Route11" color="4" fill="7" visible="no" active="no"/>
-<layer number="12" name="Route12" color="1" fill="5" visible="no" active="no"/>
-<layer number="13" name="Route13" color="4" fill="5" visible="no" active="no"/>
-<layer number="14" name="Route14" color="1" fill="6" visible="no" active="no"/>
-<layer number="15" name="Route15" color="4" fill="6" visible="no" active="no"/>
-<layer number="16" name="Bottom" color="1" fill="1" visible="no" active="no"/>
-<layer number="17" name="Pads" color="2" fill="1" visible="no" active="no"/>
-<layer number="18" name="Vias" color="2" fill="1" visible="no" active="no"/>
-<layer number="19" name="Unrouted" color="6" fill="1" visible="no" active="no"/>
-<layer number="20" name="Dimension" color="15" fill="1" visible="no" active="no"/>
-<layer number="21" name="tPlace" color="7" fill="1" visible="no" active="no"/>
-<layer number="22" name="bPlace" color="7" fill="1" visible="no" active="no"/>
-<layer number="23" name="tOrigins" color="15" fill="1" visible="no" active="no"/>
-<layer number="24" name="bOrigins" color="15" fill="1" visible="no" active="no"/>
-<layer number="25" name="tNames" color="7" fill="1" visible="no" active="no"/>
-<layer number="26" name="bNames" color="7" fill="1" visible="no" active="no"/>
-<layer number="27" name="tValues" color="7" fill="1" visible="no" active="no"/>
-<layer number="28" name="bValues" color="7" fill="1" visible="no" active="no"/>
+<layer number="1" name="Top" color="4" fill="1" visible="yes" active="no"/>
+<layer number="2" name="Route2" color="1" fill="3" visible="yes" active="no"/>
+<layer number="3" name="Route3" color="4" fill="3" visible="yes" active="no"/>
+<layer number="4" name="Route4" color="1" fill="4" visible="yes" active="no"/>
+<layer number="5" name="Route5" color="4" fill="4" visible="yes" active="no"/>
+<layer number="6" name="Route6" color="1" fill="8" visible="yes" active="no"/>
+<layer number="7" name="Route7" color="4" fill="8" visible="yes" active="no"/>
+<layer number="8" name="Route8" color="1" fill="2" visible="yes" active="no"/>
+<layer number="9" name="Route9" color="4" fill="2" visible="yes" active="no"/>
+<layer number="10" name="Route10" color="1" fill="7" visible="yes" active="no"/>
+<layer number="11" name="Route11" color="4" fill="7" visible="yes" active="no"/>
+<layer number="12" name="Route12" color="1" fill="5" visible="yes" active="no"/>
+<layer number="13" name="Route13" color="4" fill="5" visible="yes" active="no"/>
+<layer number="14" name="Route14" color="1" fill="6" visible="yes" active="no"/>
+<layer number="15" name="Route15" color="4" fill="6" visible="yes" active="no"/>
+<layer number="16" name="Bottom" color="1" fill="1" visible="yes" active="no"/>
+<layer number="17" name="Pads" color="2" fill="1" visible="yes" active="no"/>
+<layer number="18" name="Vias" color="2" fill="1" visible="yes" active="no"/>
+<layer number="19" name="Unrouted" color="6" fill="1" visible="yes" active="no"/>
+<layer number="20" name="Dimension" color="15" fill="1" visible="yes" active="no"/>
+<layer number="21" name="tPlace" color="7" fill="1" visible="yes" active="no"/>
+<layer number="22" name="bPlace" color="7" fill="1" visible="yes" active="no"/>
+<layer number="23" name="tOrigins" color="15" fill="1" visible="yes" active="no"/>
+<layer number="24" name="bOrigins" color="15" fill="1" visible="yes" active="no"/>
+<layer number="25" name="tNames" color="7" fill="1" visible="yes" active="no"/>
+<layer number="26" name="bNames" color="7" fill="1" visible="yes" active="no"/>
+<layer number="27" name="tValues" color="7" fill="1" visible="yes" active="no"/>
+<layer number="28" name="bValues" color="7" fill="1" visible="yes" active="no"/>
 <layer number="29" name="tStop" color="7" fill="3" visible="no" active="no"/>
 <layer number="30" name="bStop" color="7" fill="6" visible="no" active="no"/>
@@
 <layer number="35" name="tGlue" color="7" fill="4" visible="no" active="no"/>
 <layer number="36" name="bGlue" color="7" fill="5" visible="no" active="no"/>
-<layer number="37" name="tTest" color="7" fill="1" visible="no" active="no"/>
-<layer number="38" name="bTest" color="7" fill="1" visible="no" active="no"/>
+<layer number="37" name="tTest" color="7" fill="1" visible="yes" active="no"/>
+<layer number="38" name="bTest" color="7" fill="1" visible="yes" active="no"/>
 <layer number="39" name="tKeepout" color="4" fill="11" visible="no" active="no"/>
 <layer number="40" name="bKeepout" color="1" fill="11" visible="no" active="no"/>
@@
 <layer number="44" name="Drills" color="7" fill="1" visible="no" active="no"/>
 <layer number="45" name="Holes" color="7" fill="1" visible="no" active="no"/>
-<layer number="46" name="Milling" color="3" fill="1" visible="no" active="no"/>
-<layer number="47" name="Measures" color="7" fill="1" visible="no" active="no"/>
-<layer number="48" name="Document" color="7" fill="1" visible="no" active="no"/>
-<layer number="49" name="Reference" color="7" fill="1" visible="no" active="no"/>
-<layer number="50" name="dxf" color="7" fill="1" visible="no" active="no"/>
-<layer number="51" name="tDocu" color="7" fill="1" visible="no" active="no"/>
-<layer number="52" name="bDocu" color="7" fill="1" visible="no" active="no"/>
-<layer number="53" name="tGND_GNDA" color="7" fill="9" visible="no" active="no"/>
-<layer number="54" name="bGND_GNDA" color="1" fill="9" visible="no" active="no"/>
+<layer number="46" name="Milling" color="3" fill="1" visible="yes" active="no"/>
+<layer number="47" name="Measures" color="7" fill="1" visible="yes" active="no"/>
+<layer number="48" name="Document" color="7" fill="1" visible="yes" active="no"/>
+<layer number="49" name="Reference" color="7" fill="1" visible="yes" active="no"/>
+<layer number="50" name="dxf" color="7" fill="1" visible="yes" active="no"/>
+<layer number="51" name="tDocu" color="7" fill="1" visible="yes" active="no"/>
+<layer number="52" name="bDocu" color="7" fill="1" visible="yes" active="no"/>
+<layer number="53" name="tGND_GNDA" color="7" fill="9" visible="yes" active="no"/>
+<layer number="54" name="bGND_GNDA" color="1" fill="9" visible="yes" active="no"/>
 <layer number="91" name="Nets" color="2" fill="1" visible="yes" active="yes"/>
 <layer number="92" name="Busses" color="1" fill="1" visible="yes" active="yes"/>
@@
 <parts>
 <part name="IC3" library="lindsay-mosfet-driver" deviceset="IR2110" device=""/>
-<part name="D1" library="diode" deviceset="DIODE-" device="D-5" value="UF4004"/>
+<part name="D1" library="diode" deviceset="DIODE-" device="D-7.5" value="UF4004"/>
 <part name="C8" library="rcl" deviceset="CPOL-EU" device="E5-8.5" value="1u"/>
 <part name="C7" library="rcl" deviceset="CPOL-EU" device="E5-8.5" value="1u"/>

Commit message: layouts
Parts:
- R2, R3: device pot:TRIM_EU-LI15 -> pot:TRIM_EU-LI10
Changed lines of the file:
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@@
 <part name="IC4" library="linear" deviceset="78*" device="TV" technology="05"/>
 <part name="B1" library="rectifier" deviceset="RECTIFIER-" device="GBU4"/>
-<part name="R2" library="pot" deviceset="TRIM_EU-" device="LI15"/>
-<part name="R3" library="pot" deviceset="TRIM_EU-" device="LI15"/>
+<part name="R2" library="pot" deviceset="TRIM_EU-" device="LI10"/>
+<part name="R3" library="pot" deviceset="TRIM_EU-" device="LI10"/>
 <part name="C1" library="rcl" deviceset="CPOL-EU" device="E5-8.5" value=".1u"/>
 <part name="C2" library="rcl" deviceset="CPOL-EU" device="E5-8.5" value=".1u"/>

Commit message: layouts
Parts:
- S1: value (none) -> TL32PO; device switch:320-916 -> switch:TL32PO
Other:
- note added: "Trimmer R2 500"
- note added: "Trimmer R3 1k"
- note removed: "Trimmers 500"
Changed lines of the file:
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@@
 <part name="GND1" library="supply1" deviceset="GND" device=""/>
 <part name="GND3" library="supply1" deviceset="GND" device=""/>
-<part name="S1" library="switch" deviceset="320-916" device=""/>
 <part name="GND2" library="supply1" deviceset="GND" device=""/>
 <part name="P+2" library="supply1" deviceset="VCC" device=""/>
@@
 <part name="GND9" library="supply1" deviceset="GND" device=""/>
 <part name="C6" library="rcl" deviceset="C-EU" device="075-052X106" value="10n"/>
+<part name="S1" library="switch" deviceset="TL32PO" device=""/>
 </parts>
 <sheets>
@@
 <text x="10.16" y="139.7" size="1.778" layer="97">12 VAC in</text>
 <text x="12.7" y="101.6" size="1.778" layer="97">Rectified variac out</text>
-<text x="63.5" y="78.74" size="1.778" layer="97">Trimmers 500</text>
+<text x="63.5" y="78.74" size="1.778" layer="97">Trimmer R3 1k</text>
+<text x="55.88" y="63.5" size="1.778" layer="97">Trimmer R2 500</text>
 </plain>
 <instances>
@@
 <instance part="GND1" gate="1" x="203.2" y="58.42"/>
 <instance part="GND3" gate="1" x="177.8" y="58.42"/>
-<instance part="S1" gate="1" x="167.64" y="63.5" rot="R90"/>
 <instance part="GND2" gate="1" x="162.56" y="60.96"/>
 <instance part="P+2" gate="VCC" x="119.38" y="96.52"/>
@@
 <attribute name="VALUE" x="177.4539" y="92.9162" size="1.27" layer="96" rot="R180"/>
 </instance>
+<instance part="S1" gate="BEF1" x="167.64" y="66.04" rot="R90"/>
 </instances>
 <busses>
@@
 <wire x1="175.26" y1="81.28" x2="175.26" y2="66.04" width="0.1524" layer="91"/>
 <pinref part="IC3" gate="G$1" pin="11"/>
-<pinref part="S1" gate="1" pin="P"/>
 <wire x1="175.26" y1="66.04" x2="172.72" y2="66.04" width="0.1524" layer="91"/>
+<pinref part="S1" gate="BEF1" pin="P"/>
 </segment>
 </net>
@@
 <pinref part="IC1" gate="G$1" pin="VCC+"/>
 <wire x1="119.38" y1="93.98" x2="119.38" y2="86.36" width="0.1524" layer="91"/>
-</segment>
-<segment>
-<pinref part="S1" gate="1" pin="S"/>
-<pinref part="P+1" gate="VCC" pin="VCC"/>
 </segment>
 <segment>
@@
 <junction x="109.22" y="99.06"/>
 <pinref part="P+5" gate="VCC" pin="VCC"/>
+</segment>
+<segment>
+<pinref part="P+1" gate="VCC" pin="VCC"/>
+<pinref part="S1" gate="BEF1" pin="S"/>
 </segment>
 </net>
@@
 </segment>
 <segment>
-<pinref part="S1" gate="1" pin="O"/>
-<pinref part="GND2" gate="1" pin="GND"/>
-</segment>
-<segment>
 <pinref part="IC1" gate="G$1" pin="GND"/>
 <pinref part="GND4" gate="1" pin="GND"/>
@@
 <wire x1="132.08" y1="60.96" x2="132.08" y2="66.04" width="0.1524" layer="91"/>
 </segment>
-</net>
+<segment>
+<pinref part="GND2" gate="1" pin="GND"/>
+<pinref part="S1" gate="BEF1" pin="O"/>
+</segment>
+</net>
