File: eagle/disruptor/generator.sch (EAGLE design)
At the start: 29 parts, among them IC1 NE555, IC2 74ALS04N, IC3 IR2110, IC4 7805TV, J1 PIN2F061.100, J2 PIN2F061.100, J3 PIN2F061.100, J4 PIN2F061.100, J5 PIN2F061.100, J6 PIN2F061.100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

Commit message: pre-round 2
Parts:
- removed R6, R7: 1M, rcl:R-US_0207/10
- added C10, C13, C9: (no value), resistor:CPOL-USE7.5-18
- added C11, C12: 2200, resistor:CPOL-USE10-35
- added C14, C15: 560u, rcl:CPOL-EUE7.5-16
- added D2, D3: (no value), diode:ZENER-DIODEZD-10
- C1: value .1u -> .01u
- C7: value 1u -> min 12 nF
- R4, R5: value 100 -> 10
- RA, RB: value (none) -> 10k
- renumbered R2 to RB, R3 to RA
Connections:
- removed net N$13: J5.1, Q1.D
- removed net TRANS1: C7.-, IC3.5, J1.1, Q1.S, R6.2
- removed net TRANS2: J2.1, Q2.D
- new net N$6: C11.+, C12.+, C14.+, J5.1, Q1.D
- new net N$8: C14.-, C15.+, J2.1
- new net TRANS: C7.-, D2.A, IC3.5, J1.1, Q1.S, Q2.D
- net GND: now also C10.-, C11.-, C12.-, C13.-, C15.-, C9.-, D3.A; no longer R7.2
- net N$11: now also D3.C; no longer R7.1
- net N$12: now also D2.C; no longer R6.1
- net VDD: now also C10.+, C13.+, C9.+
Other:
- moved on the sheet: J2
