File: eagle/disruptor/caps.sch (EAGLE design)
At the start: 18 parts, among them IC5 7812TV, J1 PIN2F061.100, J2 PIN2F061.100, J3 PIN2F061.100, J4 PIN2F061.100, J5 PIN2F061.100, J6 PIN2F061.100, Q1 2N5883, T1 2N3055, T2 2N3055

Commit message: rev2
Parts:
- removed C3, C4: 1u, rcl:CPOL-EUE10-20
- removed IC5: 7812TV, linear:7812TV
- removed J5, J6: PIN2F061.100, con-faston:PIN2F061.100
- removed Q1: 2N5883, transistor-pnp:2N4905
- removed R1: 1K, rcl:R-US_0207/15
- removed R2: 1.8K, rcl:R-US_0207/15
- removed R3: 10, rcl:R-US_0207/15
- removed R4: 1, rcl:R-US_0922/22
- removed T1, T2: 2N3055, transistor:2N3055
- removed X2, X3: (no value), con-ptr500:AK300/8
- added C1, C2: (no value), rcl:CPOL-USE10-35
Connections:
- removed net GND: C3.-, C4.-, J4.1, R2.1, X2-2.KL, X2-4.KL, X2-6.KL, X2-8.KL, X3-2.KL, X3-4.KL, X3-6.KL, X3-8.KL
- removed net N$4: IC5.VI, Q1.B, R3.2
- removed net N$5: IC5.GND, R1.1, R2.2
- removed net TEC1: J2.1, X2-1.KL, X2-3.KL
- removed net TEC2: J6.1, X2-5.KL, X2-7.KL
- removed net VDD: C4.+, IC5.VO, J1.1, J5.1, R1.2, R4.2, T1.E, T2.E, X3-1.KL, X3-3.KL, X3-5.KL, X3-7.KL
- removed net VIN: C3.+, J3.1, Q1.E, R3.1, T1.C, T2.C
- new net N$2: C1.-, C2.-, J2.1, J4.1
- net N$1: now also C1.+, C2.+, J1.1, J3.1; no longer Q1.C, R4.1, T1.B, T2.B
Other:
- note removed: "Fans out"
- note removed: "Relay"
- note removed: "TEC out"
- note removed: "Ultrasonic transducer driver"
- moved on the sheet: J1, J2, J3, J4
