File: eagle/disruptor/generator2.sch (EAGLE design)
At the start: 29 parts, among them IC1 NE555, IC2 74ALS04N, IC3 IR2110, IC4 7805TV, J1 PIN2F061.100, J2 PIN2F061.100, J3 PIN2F061.100, J4 PIN2F061.100, J5 PIN2F061.100, J6 PIN2F061.100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

Commit message: rev2
Parts:
- added B2: RECTIFIER-GBU4, rectifier:RECTIFIER-GBU4
- added C10, C11, C12, C9: (no value), resistor:CPOL-USE7.5-18
- D1: device diode:DIODE-D-5 -> diode:DIODE-D-7.5
- R2, R3: device pot:TRIM_EU-LI15 -> pot:TRIM_EU-LI10
- R4, R5: value (none) -> 100
- R6, R7: value (none) -> 1M
- S1: value (none) -> TL32PO; device switch:320-916 -> switch:TL32PO
Connections:
- net N$14 renamed LIN
- net N$15 renamed TRANS2
- net N$4 renamed HIN
- net N$5 renamed LO
- net N$6 renamed TRANS1
- net N$8 renamed HO
- removed net N$13: J5.1, Q1.D
- new net N$4: B2.AC1, J5.1
- new net N$5: B2.AC2, J6.1
- new net N$6: B2.+, C11.+, C12.+, Q1.D
- net GND: now also B2.-, C10.-, C11.-, C12.-, C9.-; no longer J6.1
- net VDD: now also C10.+, C9.+
Other:
- note added: "Trimmer R2 500"
- note added: "Trimmer R3 1k"
- note removed: "Trimmers 500"
- moved on the sheet: J2
