File: eagle/disruptor/generator3.sch (EAGLE design)
At the start: 35 parts, among them IC1 NE555, IC2 74ALS04N, IC3 IR2110, IC4 7805TV, J1 PIN2F061.100, J2 PIN2F061.100, J3 PIN2F061.100, J4 PIN2F061.100, J5 PIN2F061.100, J6 PIN2F061.100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

Commit message: gen4
Connections:
- net TRANS2 renamed TRANS
Changed lines of the file:
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@@
 </segment>
 </net>
-<net name="TRANS2" class="0">
+<net name="TRANS" class="0">
 <segment>
 <pinref part="Q2" gate="G$1" pin="D"/>
