File: eagle/disruptor/generator3.sch (EAGLE design)
At the start: 35 parts, among them IC1 NE555, IC2 74ALS04N, IC3 IR2110, IC4 7805TV, J1 PIN2F061.100, J2 PIN2F061.100, J3 PIN2F061.100, J4 PIN2F061.100, J5 PIN2F061.100, J6 PIN2F061.100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

Commit message: generator 4 is the correct way.
Parts:
- C7: value 1u -> min 12nF
- R4, R5: value 100 -> 10
Changed lines of the file:
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@@
 <part name="D1" library="diode" deviceset="DIODE-" device="D-7.5" value="UF4004"/>
 <part name="C8" library="rcl" deviceset="CPOL-EU" device="E5-8.5" value="1u"/>
-<part name="C7" library="rcl" deviceset="CPOL-EU" device="E5-8.5" value="1u"/>
+<part name="C7" library="rcl" deviceset="CPOL-EU" device="E5-8.5" value="min 12nF"/>
 <part name="FRAME1" library="frames" deviceset="A4L-LOC" device=""/>
 <part name="IC1" library="st-microelectronics" deviceset="NE555" device=""/>
@@
 <part name="C5" library="rcl" deviceset="CPOL-EU" device="E5-8.5" value="1u"/>
 <part name="GND8" library="supply1" deviceset="GND" device=""/>
-<part name="R4" library="rcl" deviceset="R-US_" device="0207/10" value="100"/>
-<part name="R5" library="rcl" deviceset="R-US_" device="0207/10" value="100"/>
+<part name="R4" library="rcl" deviceset="R-US_" device="0207/10" value="10"/>
+<part name="R5" library="rcl" deviceset="R-US_" device="0207/10" value="10"/>
 <part name="J1" library="con-faston" deviceset="PIN2" device="F061.100"/>
 <part name="J2" library="con-faston" deviceset="PIN2" device="F061.100"/>
