File: eagle/disruptor/generator3.brd (EAGLE design)
At the start: 126.5 x 120.7 mm, 35 parts, among them IC1 NE555, IC2 74ALS04N, IC3 IR2110, IC4 7805TV, J1 PIN2F061.100, J2 PIN2F061.100, J3 PIN2F061.100, J4 PIN2F061.100, J5 PIN2F061.100, J6 PIN2F061.100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

Commit message: gen3
Parts:
- moved R7 0.25 mm to (18.3, 5.08)
Connections:
- removed net TRANS1: C7.-, IC3.5, J1.A1, J1.A2, Q1.S, R6.2
- net GND: now also J2.A1, J2.A2
- net TRANS2: now also C7.-, IC3.5, J1.A1, J1.A2, Q1.S, R6.2; no longer J2.A1, J2.A2
Routing:
- net TRANS1: track 168.1 -> 0.00 mm
- net TRANS2: track 69.8 -> 14.5 mm

Commit message: gen4
Parts:
- moved J1 2.34 mm to (69.1, 19.1)
Connections:
- net TRANS2 renamed TRANS
Routing:
- net TRANS: track 14.5 -> 207.0 mm
Changed lines of the file:
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@@
 <element name="R4" library="rcl" package="0207/10" value="100" x="45.72" y="29.21"/>
 <element name="R5" library="rcl" package="0207/10" value="100" x="50.8" y="10.16" rot="R90"/>
-<element name="J1" library="con-faston" package="F061.100" value="PIN2F061.100" x="68.58" y="21.336" rot="R180">
-<attribute name="OC_NEWARK" value="unknown" x="68.58" y="21.336" size="1.778" layer="27" rot="R180" display="off"/>
-<attribute name="MPN" value="" x="68.58" y="21.336" size="1.778" layer="27" rot="R180" display="off"/>
-<attribute name="MF" value="" x="68.58" y="21.336" size="1.778" layer="27" rot="R180" display="off"/>
-<attribute name="OC_FARNELL" value="unknown" x="68.58" y="21.336" size="1.778" layer="27" rot="R180" display="off"/>
+<element name="J1" library="con-faston" package="F061.100" value="PIN2F061.100" x="69.088" y="19.05" rot="R180">
+<attribute name="OC_NEWARK" value="unknown" x="69.088" y="19.05" size="1.778" layer="27" rot="R180" display="off"/>
+<attribute name="MPN" value="" x="69.088" y="19.05" size="1.778" layer="27" rot="R180" display="off"/>
+<attribute name="MF" value="" x="69.088" y="19.05" size="1.778" layer="27" rot="R180" display="off"/>
+<attribute name="OC_FARNELL" value="unknown" x="69.088" y="19.05" size="1.778" layer="27" rot="R180" display="off"/>
 </element>
 <element name="J2" library="con-faston" package="F061.100" value="PIN2F061.100" x="68.58" y="5.588" rot="R180">
@@
 <contactref element="J2" pad="A1"/>
 <contactref element="J2" pad="A2"/>
+<wire x1="60.198" y1="63.5" x2="60.198" y2="71.12" width="0" layer="19" extent="1-1"/>
 </signal>
 <signal name="VCC">
@@
 <wire x1="36.576" y1="29.21" x2="40.64" y2="29.21" width="1.6764" layer="1"/>
 </signal>
-<signal name="TRANS2">
+<signal name="TRANS">
 <contactref element="Q2" pad="D"/>
 <contactref element="IC3" pad="5"/>
@@
 <contactref element="J1" pad="A2"/>
 <wire x1="22.098" y1="19.05" x2="36.576" y2="19.05" width="1.6764" layer="1"/>
-<wire x1="52.578" y1="71.12" x2="52.578" y2="80.01" width="0" layer="19" extent="1-1"/>
-<wire x1="66.08" y1="21.336" x2="52.578" y2="71.12" width="0" layer="19" extent="1-1"/>
-<wire x1="71.08" y1="21.336" x2="66.08" y2="21.336" width="0" layer="19" extent="1-1"/>
-<wire x1="36.576" y1="19.05" x2="66.08" y2="21.336" width="0" layer="19" extent="1-1"/>
-<wire x1="36.068" y1="7.62" x2="36.576" y2="19.05" width="0" layer="19" extent="1-1"/>
+<wire x1="52.578" y1="80.01" x2="52.578" y2="77.47" width="2.54" layer="1"/>
+<wire x1="36.576" y1="19.05" x2="31.75" y2="19.05" width="1.6764" layer="1"/>
+<wire x1="31.75" y1="19.05" x2="31.75" y2="7.62" width="1.6764" layer="1"/>
+<wire x1="31.75" y1="7.62" x2="37.084" y2="7.62" width="1.6764" layer="1"/>
+<wire x1="52.578" y1="70.358" x2="52.578" y2="77.47" width="1.6764" layer="1"/>
+<wire x1="71.12" y1="74.93" x2="71.12" y2="20.828" width="2.54" layer="1"/>
+<wire x1="36.576" y1="19.05" x2="56.134" y2="19.05" width="2.54" layer="1"/>
+<wire x1="56.134" y1="19.05" x2="66.588" y2="19.05" width="2.54" layer="1"/>
+<wire x1="71.12" y1="74.93" x2="53.086" y2="74.93" width="2.54" layer="1"/>
+<wire x1="66.588" y1="19.05" x2="74.168" y2="19.05" width="1.6764" layer="1"/>
+<wire x1="74.168" y1="19.05" x2="74.168" y2="21.082" width="1.6764" layer="1"/>
+<wire x1="74.168" y1="21.082" x2="63.754" y2="21.082" width="1.6764" layer="1"/>
+<wire x1="63.754" y1="21.082" x2="63.5" y2="20.828" width="1.6764" layer="1"/>
+<wire x1="63.5" y1="20.828" x2="63.5" y2="17.018" width="1.6764" layer="1"/>
+<wire x1="63.5" y1="17.018" x2="74.168" y2="17.018" width="1.6764" layer="1"/>
+<wire x1="74.168" y1="17.018" x2="74.168" y2="19.304" width="1.6764" layer="1"/>
+<wire x1="74.168" y1="19.304" x2="73.914" y2="19.558" width="1.6764" layer="1"/>
+<wire x1="73.914" y1="19.558" x2="64.77" y2="19.558" width="1.6764" layer="1"/>
+<wire x1="64.77" y1="19.558" x2="64.262" y2="20.066" width="1.6764" layer="1"/>
+<wire x1="64.262" y1="20.066" x2="64.262" y2="18.034" width="1.6764" layer="1"/>
+<wire x1="64.262" y1="18.034" x2="64.516" y2="17.78" width="1.6764" layer="1"/>
+<wire x1="64.516" y1="17.78" x2="73.914" y2="17.78" width="1.6764" layer="1"/>
+<wire x1="52.578" y1="70.358" x2="52.578" y2="71.12" width="0" layer="19" extent="1-1"/>
+<wire x1="53.086" y1="74.93" x2="52.578" y2="77.47" width="0" layer="19" extent="1-1"/>
+<wire x1="71.588" y1="19.05" x2="71.12" y2="20.828" width="0" layer="19" extent="1-1"/>
+<wire x1="73.914" y1="19.558" x2="71.588" y2="19.05" width="0" layer="19" extent="1-1"/>
+<wire x1="36.068" y1="7.62" x2="37.084" y2="7.62" width="0" layer="19" extent="1-1"/>
 </signal>
 <signal name="N$3">

Commit message: gen4b
Parts:
- R6, R7: value 1M -> 22k
Changed lines of the file:
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@@
 <attribute name="OC_FARNELL" value="unknown" x="-40.386" y="86.868" size="1.778" layer="27" display="off"/>
 </element>
-<element name="R6" library="rcl" package="0207/10" value="1M" x="36.576" y="24.13" rot="R270"/>
-<element name="R7" library="rcl" package="0207/10" value="1M" x="18.288" y="5.08" rot="R180"/>
+<element name="R6" library="rcl" package="0207/10" value="22k" x="36.576" y="24.13" rot="R270"/>
+<element name="R7" library="rcl" package="0207/10" value="22k" x="18.288" y="5.08" rot="R180"/>
 <element name="C3" library="rcl" package="C075-052X106" value="10n" x="29.972" y="64.77" rot="R180"/>
 <element name="C6" library="rcl" package="C075-052X106" value="10n" x="53.848" y="42.926" rot="R180"/>

Commit message: generator 4 is the correct way.
Parts:
- C7: value 1u -> min 12nF
- R4, R5: value 100 -> 10
Changed lines of the file:
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@@
 <element name="D1" library="diode" package="D-7.5" value="UF4004" x="57.658" y="88.9"/>
 <element name="C8" library="rcl" package="E5-8,5" value="1u" x="61.468" y="82.296" rot="R270"/>
-<element name="C7" library="rcl" package="E5-8,5" value="1u" x="50.038" y="80.01"/>
+<element name="C7" library="rcl" package="E5-8,5" value="min 12nF" x="50.038" y="80.01"/>
 <element name="IC1" library="st-microelectronics" package="DIL-08" value="NE555" x="17.018" y="59.69">
 <attribute name="OC_NEWARK" value="89K1486" x="76.708" y="-11.43" size="1.778" layer="27" display="off"/>
@@
 <element name="C4" library="rcl" package="E5-8,5" value="1u" x="67.818" y="112.014" rot="R270"/>
 <element name="C5" library="rcl" package="E5-8,5" value="1u" x="67.818" y="99.06" rot="R90"/>
-<element name="R4" library="rcl" package="0207/10" value="100" x="45.72" y="29.21"/>
-<element name="R5" library="rcl" package="0207/10" value="100" x="50.8" y="10.16" rot="R90"/>
+<element name="R4" library="rcl" package="0207/10" value="10" x="45.72" y="29.21"/>
+<element name="R5" library="rcl" package="0207/10" value="10" x="50.8" y="10.16" rot="R90"/>
 <element name="J1" library="con-faston" package="F061.100" value="PIN2F061.100" x="69.088" y="19.05" rot="R180">
 <attribute name="OC_NEWARK" value="unknown" x="69.088" y="19.05" size="1.778" layer="27" rot="R180" display="off"/>
