File: eagle/disruptor/generator4.brd (EAGLE design)
At the start: 126.5 x 120.7 mm, 37 parts, among them IC1 NE555, IC2 74ALS04N, IC3 IR2110, IC4 7805TV, J1 PIN2F061.100, J2 PIN2F061.100, J3 PIN2F061.100, J4 PIN2F061.100, J5 PIN2F061.100, J6 PIN2F061.100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

Commit message: gen 4 board layout done.
Parts:
- removed B2: RECTIFIER-GBU4, rectifier:GBU4
- C14, C15: value 50u -> 470u; device rcl:E5-8,5 -> rcl:E7,5-16
- moved J6 53.6 mm to (-41.4, 33.3)
- moved C15 35.8 mm to (20.8, 8.89)
- moved R7 29.1 mm to (10.2, 33.0)
- moved R5 28.5 mm to (24.6, 28.4)
- moved J5 23.9 mm to (-41.4, 47.8)
- moved Q2 21.4 mm to (12.7, 21.6), turned to 180 degrees
- moved C12 20.9 mm to (-27.2, 69.6), turned to 90 degrees
- moved Q1 16.5 mm to (41.1, 21.8), turned to 180 degrees
- moved R6 9.37 mm to (38.6, 33.3), turned to 180 degrees
- moved R4 7.89 mm to (53.6, 28.7), turned to 90 degrees
- moved C11 7.27 mm to (-16.3, 20.1), turned to 270 degrees
- moved C14 6.93 mm to (49.8, 9.14)
- moved J1 5.21 mm to (69.1, 19.4)
- moved J2 1.37 mm to (69.1, 4.32)
Connections:
- removed net N$4: B2.AC1, J5.A1, J5.A2
- removed net N$5: B2.AC2, J6.A1, J6.A2
- net GND: now also J6.A1, J6.A2; no longer B2.-
- net N$6: now also J5.A1, J5.A2; no longer B2.+
Routing:
- net TRANS: track 27.7 -> 221.4 mm
- net N$8: track 0.00 -> 95.7 mm
- net LO: track 1.52 -> 95.1 mm
- net N$6: track 77.6 -> 149.6 mm
- net N$5: track 63.4 -> 0.00 mm
- net N$4: track 60.3 -> 0.00 mm
- net N$12: track 0.00 -> 19.6 mm
- net HO: track 54.9 -> 69.6 mm
- net N$11: track 6.60 -> 19.1 mm

Commit message: final board
Routing:
- net N$8: track 95.7 -> 99.3 mm
- net TRANS: track 221.4 -> 223.1 mm
Changed lines of the file:
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@@
 <wire x1="52.578" y1="80.01" x2="52.578" y2="77.47" width="2.54" layer="1"/>
 <wire x1="52.578" y1="70.358" x2="52.578" y2="77.47" width="1.6764" layer="1"/>
-<wire x1="73.152" y1="74.93" x2="53.086" y2="74.93" width="2.54" layer="1"/>
+<wire x1="73.8124" y1="75.0062" x2="53.086" y2="74.93" width="2.54" layer="1"/>
 <wire x1="71.5626" y1="19.431" x2="73.152" y2="19.812" width="2.54" layer="1"/>
-<wire x1="73.152" y1="19.812" x2="73.152" y2="20.066" width="2.54" layer="1"/>
-<wire x1="73.152" y1="20.066" x2="73.152" y2="74.93" width="2.54" layer="1"/>
+<wire x1="73.152" y1="19.812" x2="73.7362" y2="19.939" width="2.54" layer="1"/>
+<wire x1="73.7362" y1="19.939" x2="73.8124" y2="75.0062" width="2.54" layer="1"/>
 <wire x1="38.608" y1="24.384" x2="38.608" y2="28.448" width="1.6764" layer="1"/>
 <wire x1="38.608" y1="28.448" x2="33.528" y2="33.274" width="1.6764" layer="1"/>
@@
 <wire x1="64.516" y1="17.6022" x2="64.516" y2="20.32" width="1.6764" layer="1"/>
 <wire x1="64.516" y1="20.32" x2="72.898" y2="20.32" width="1.6764" layer="1"/>
-<wire x1="72.898" y1="20.32" x2="73.152" y2="20.066" width="1.6764" layer="1"/>
+<wire x1="72.898" y1="20.32" x2="73.7362" y2="19.939" width="1.6764" layer="1"/>
 <wire x1="66.5626" y1="19.431" x2="66.802" y2="19.558" width="1.6764" layer="1"/>
 <wire x1="66.802" y1="19.558" x2="68.072" y2="18.288" width="1.6764" layer="1"/>
@@
 <wire x1="65.024" y1="5.842" x2="66.588" y2="4.318" width="2.54" layer="1"/>
 <wire x1="66.588" y1="4.318" x2="72.898" y2="4.318" width="2.54" layer="1"/>
-<wire x1="66.588" y1="4.318" x2="74.168" y2="4.318" width="1.6764" layer="1"/>
+<wire x1="72.898" y1="4.318" x2="74.168" y2="4.318" width="1.6764" layer="1"/>
 <wire x1="74.168" y1="4.318" x2="74.168" y2="6.35" width="1.6764" layer="1"/>
 <wire x1="74.168" y1="6.35" x2="72.39" y2="6.35" width="1.6764" layer="1"/>
@@
 <wire x1="63.5" y1="6.35" x2="72.39" y2="6.35" width="1.6764" layer="1"/>
 <wire x1="72.39" y1="6.35" x2="72.898" y2="5.842" width="1.6764" layer="1"/>
-<wire x1="72.898" y1="4.318" x2="71.588" y2="4.318" width="0" layer="19" extent="1-1"/>
 <wire x1="24.638" y1="8.89" x2="24.638" y2="9.398" width="0" layer="19" extent="1-1"/>
+<wire x1="72.898" y1="4.318" x2="64.7446" y2="4.318" width="1.6764" layer="1"/>
+<wire x1="64.7446" y1="4.318" x2="64.7446" y2="3.8354" width="1.6764" layer="1"/>
+<wire x1="64.7446" y1="3.8354" x2="65.6336" y2="3.8354" width="1.6764" layer="1"/>
+<wire x1="65.6336" y1="3.8354" x2="65.6336" y2="3.5052" width="1.6764" layer="1"/>
+<wire x1="65.6336" y1="3.5052" x2="71.588" y2="4.318" width="0" layer="19" extent="1-16"/>
 </signal>
 </signals>

Commit message: beefier cap values
Parts:
- C11, C12: value (none) -> 2200
- C14, C15: value 470u -> 560u
Changed lines of the file:
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@@
 <element name="C9" library="resistor" package="E7,5-18" value="" x="41.402" y="106.934" rot="R90"/>
 <element name="C10" library="resistor" package="E7,5-18" value="" x="19.558" y="106.934" rot="R90"/>
-<element name="C11" library="resistor" package="EB35D" value="" x="-16.256" y="20.066" rot="R270"/>
-<element name="C12" library="resistor" package="EB35D" value="" x="-27.178" y="69.596" rot="R90"/>
+<element name="C11" library="resistor" package="EB35D" value="2200" x="-16.256" y="20.066" rot="R270"/>
+<element name="C12" library="resistor" package="EB35D" value="2200" x="-27.178" y="69.596" rot="R90"/>
 <element name="C13" library="resistor" package="E7,5-18" value="" x="-2.286" y="106.934" rot="R90"/>
-<element name="C14" library="rcl" package="E7,5-16" value="470u" x="49.784" y="9.144"/>
-<element name="C15" library="rcl" package="E7,5-16" value="470u" x="20.828" y="8.89" rot="R180"/>
+<element name="C14" library="rcl" package="E7,5-16" value="560u" x="49.784" y="9.144"/>
+<element name="C15" library="rcl" package="E7,5-16" value="560u" x="20.828" y="8.89" rot="R180"/>
 </elements>
 <signals>
