File: eagle/disruptor/generator_cd4047.brd (EAGLE design)
At the start: 126.5 x 120.7 mm, 36 parts, among them IC1 NE555, IC2 74ALS04N, IC3 IR2110, IC4 7805TV, J1 PIN2F061.100, J2 PIN2F061.100, J3 PIN2F061.100, J4 PIN2F061.100, J5 PIN2F061.100, J6 PIN2F061.100, Q1 STP11NM60, Q2 STP11NM60

Commit message: wryqedx
Parts:
- removed IC1: NE555, st-microelectronics:DIL-08
- removed IC2: 74ALS04N, 74xx-eu:DIL14
- removed RA, RB: 10k, pot:LI10
- added IC5: 4047N, 40xx:DIL14
- added R3: 500k, pot:RJ9W
- C1: value .01u -> 50p; device rcl:E5-8,5 -> rcl:C075-042X103
- C3: device rcl:C075-052X106 -> rcl:C075-042X103
- IC4: value 7805TV -> 7812TV
- R5: device rcl:0207/10 -> rcl:0207/15
- moved D1 48.1 mm to (47.6, 41.8), turned to 180 degrees
- moved S1 34.7 mm to (57.9, 85.0), turned to 0 degrees
- moved C6 33.0 mm to (51.4, 75.9), turned to 0 degrees
- moved C7 29.6 mm to (50.2, 50.4), turned to 180 degrees
- moved C2 28.0 mm to (5.87, 84.6), turned to 270 degrees
- moved C8 21.6 mm to (39.9, 84.3)
- moved C3 21.1 mm to (19.9, 83.3), turned to 270 degrees
- moved C1 15.1 mm to (16.7, 64.7), turned to 0 degrees
- moved IC3 9.15 mm to (46.4, 64.6), turned to 0 degrees
- moved R5 6.28 mm to (25.0, 34.2)
- moved R4 3.20 mm to (59.1, 29.5)
Connections:
- removed net GND: B1.-, C1.-, C10.-, C11.-, C12.-, C13.-, C15.-, C2.-, C3.1, C4.-, C5.-, C6.1, C8.-, C9.-, IC1.1, IC2.7, IC3.13, IC3.2, IC4.2, J6.A1, J6.A2, Q2.S, R2.2, S1.1
- removed net LIN: IC2.4, IC3.12
- removed net VCC: C2.+, C5.+, C6.2, IC1.4, IC1.8, IC2.14, IC3.9, IC4.3, RA.E, S1.3
- new net N$14: IC3.10, IC5.11
- new net VSS: B1.-, C10.-, C11.-, C12.-, C13.-, C15.-, C2.-, C3.2, C4.-, C5.-, C6.1, C8.-, C9.-, IC3.13, IC3.2, IC4.2, IC5.12, IC5.7, IC5.8, IC5.9, J6.A1, J6.A2, Q2.S, R2.2, S1.1
- net N$2: now also IC5.2, R3.A, R3.S; no longer C1.+, IC1.2, IC1.6, RB.A, RB.S
- net N$3: now also C1.1, IC5.3, R3.E; no longer C3.2, IC1.5
- net N$4: now also C1.2, IC5.1; no longer IC1.3, IC2.1
- net N$5: now also IC3.12, IC5.10; no longer IC2.2, IC2.3, IC3.10
- net N$7: now also B1.+, C10.+, C13.+, C4.+, C9.+, IC4.1; no longer IC1.7, RA.A, RA.S, RB.E
- net VDD: now also C2.+, C3.1, C5.+, C6.2, IC3.9, IC4.3, IC5.14, IC5.4, IC5.5, IC5.6, S1.3; no longer B1.+, C10.+, C13.+, C4.+, C9.+, IC4.1
Routing:
- net VCC: track 219.9 -> 0.00 mm
- net LO: track 95.1 -> 24.6 mm, vias 2 -> 0
- net N$7: track 34.1 -> 97.6 mm
- net TRANS: track 171.5 -> 112.5 mm, vias 2 -> 0
- net VDD: track 158.3 -> 215.9 mm
- net LIN: track 53.9 -> 0.00 mm, vias 2 -> 0
- net GND: track 52.4 -> 0.00 mm
- net N$14: track 0.00 -> 48.9 mm
- net HO: track 64.9 -> 28.4 mm, vias 2 -> 0
- net N$2: track 54.9 -> 21.3 mm, vias 2 -> 0
- net N$3: track 7.87 -> 18.8 mm
- net N$5: track 44.4 -> 53.2 mm, vias 1 -> 0
- net N$17: track 15.0 -> 21.4 mm
- net N$1: track 24.2 -> 19.9 mm
- net N$4: track 14.0 -> 10.0 mm
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- added copper zone on layer 1, net VSS
- added copper zone on layer 16, net VSS
- removed copper zone on layer 1, net GND
- removed copper zone on layer 16, net GND
