File: eagle/disruptor/generator_cd4047.sch (EAGLE design)
At the start: 36 parts, among them IC1 NE555, IC2 74ALS04N, IC3 IR2110, IC4 7805TV, J1 PIN2F061.100, J2 PIN2F061.100, J3 PIN2F061.100, J4 PIN2F061.100, J5 PIN2F061.100, J6 PIN2F061.100, Q1 STP11NM60, Q2 STP11NM60

Commit message: wryqedx
Parts:
- removed IC1: NE555, st-microelectronics:NE555
- removed IC2: 74ALS04N, 74xx-eu:74ALS04N
- removed RA, RB: 10k, pot:TRIM_EU-LI10
- added IC5: 4047N, 40xx:4047N
- added R3: 500k, pot:TRIM_US-RJ9W
- C1: value .01u -> 50p; device rcl:CPOL-EUE5-8.5 -> rcl:C-US075-042X103
- C3: device rcl:C-EU075-052X106 -> rcl:C-US075-042X103
- IC4: value 7805TV -> 7812TV; device linear:7805TV -> linear:7812TV
- R5: device rcl:R-US_0207/10 -> rcl:R-US_0207/15
Connections:
- removed net GND: B1.-, C1.-, C10.-, C11.-, C12.-, C13.-, C15.-, C2.-, C3.1, C4.-, C5.-, C6.1, C8.-, C9.-, IC1.GND, IC3.13, IC3.2, IC4.GND, J6.1, Q2.S, R2.2, S1.O
- removed net LIN: IC2B.O, IC3.12
- removed net VCC: C2.+, C5.+, C6.2, IC1./RES, IC1.VCC+, IC3.9, IC4.VO, RA.E, S1.S
- new net N$14: IC3.10, IC5A.!Q
- new net VSS: B1.-, C10.-, C11.-, C12.-, C13.-, C15.-, C2.-, C3.2, C4.-, C5.-, C6.1, C8.-, C9.-, IC3.13, IC3.2, IC4.GND, IC5A.+T, IC5A.RES, IC5A.RET, J6.1, Q2.S, R2.2, S1.O
- net N$2: now also IC5A.R, R3.A, R3.S; no longer C1.+, IC1.TRE, IC1.TRI, RB.A, RB.S
- net N$3: now also C1.1, IC5A.R/C, R3.E; no longer C3.2, IC1.CON
- net N$4: now also C1.2, IC5A.C; no longer IC1.OUT, IC2A.I
- net N$5: now also IC3.12, IC5A.Q; no longer IC2A.O, IC2B.I, IC3.10
- net N$7: now also B1.+, C10.+, C13.+, C4.+, C9.+, IC4.VI; no longer IC1.DIS, RA.A, RA.S, RB.E
- net VDD: now also C2.+, C3.1, C5.+, C6.2, IC3.9, IC4.VO, IC5A.!AST, IC5A.-T, IC5A.AST, S1.S; no longer B1.+, C10.+, C13.+, C4.+, C9.+, IC4.VI
Other:
- note removed: "Trimmer R3 1k"
- moved on the sheet: C2, C3
